Commit message: added second joint

File: pendulum.urdf (robot description, URDF)
Before this commit: robot pendulum, 4 links, 3 joints
Links:
- added link link_2, mass 0; visual cylinder length=0.8 radius=0.01
Joints:
- added joint joint_2: type revolute, parent link_1, child link_2, origin xyz=0.0 0 0.8 rpy=0 0 0, axis 0 1 0, limit effort=0 velocity=0
- joint joint_eef: parent link_1 -> link_2
- joint world_to_base: origin xyz=0 0 1.5 rpy=0 0 0 -> xyz=0 0 2 rpy=0 0 0

Commit message: planar robot go to cartesian via inverse jacobian

File: pendulum.urdf (robot description, URDF)
Before this commit: robot pendulum, 5 links, 4 joints
Links:
- link link_1: geometry visual cylinder length=0.5 radius=0.01
- link link_2: geometry visual cylinder length=0.5 radius=0.01
Joints:
- joint joint_2: origin xyz=0.0 0 0.8 rpy=0 0 0 -> xyz=0.0 0 0.5 rpy=0 0 0
- joint joint_eef: origin xyz=0 0 0.8 rpy=0 0 0 -> xyz=0 0 0.5 rpy=0 0 0
- joint world_to_base: origin xyz=0 0 2 rpy=0 0 0 -> xyz=0 0 1.5 rpy=0 0 0
